File: Accelerometer/BELM_Accelerometer.kicad_pcb (KiCad board)
At the start: 4 copper layers, 63.5 x 41.3 mm, 47 parts, among them J1 RJ45, U1 LIS344ALH, U2 MIC5504-3.3, U3 TSV914IPT, U4 ADS8864, U5 ADS8864, U6 ADS8864, U7 MAX6126B30+, U8 DS90LV017ATMX/NOPB, U9 SN65LVDT34D

Commit message: Fiducials
Parts:
- added REF**: Fiducial_1mm_Dia_2mm_Outer, Fiducials:Fiducial_1mm_Dia_2mm_Outer, F.Cu at (157.5, 82.5)
- added REF**: Fiducial_1mm_Dia_2mm_Outer, Fiducials:Fiducial_1mm_Dia_2mm_Outer, F.Cu at (143.5, 115.6)
- added REF**: Fiducial_1mm_Dia_2mm_Outer, Fiducials:Fiducial_1mm_Dia_2mm_Outer, F.Cu at (129.5, 82.5)
Changed lines of the file:
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@@
-(kicad_pcb (version 4) (host pcbnew 4.0.6)
+(kicad_pcb (version 4) (host pcbnew 4.0.7)
   (general
-    (links 128)
+    (links 0)
     (no_connects 0)
-    (area 107.287288 60.8 199.925715 120.772)
+    (area 96.873288 60.165 189.511715 120.137)
     (thickness 1.5748)
     (drawings 16)
     (tracks 434)
     (zones 0)
-    (modules 47)
+    (modules 50)
     (nets 40)
   )
@@
   (layers
     (0 F.Cu signal)
-    (1 In1.Cu power)
-    (2 In2.Cu power)
+    (1 In1.Cu power hide)
+    (2 In2.Cu power hide)
     (31 B.Cu signal)
     (32 B.Adhes user)
@@
     (38 B.Mask user)
     (39 F.Mask user)
-    (40 Dwgs.User user)
+    (40 Dwgs.User user hide)
     (41 Cmts.User user)
     (42 Eco1.User user)
@@
     (uvia_drill 0.1016)
   )
+  (module Fiducials:Fiducial_1mm_Dia_2mm_Outer (layer F.Cu)
+    (at 157.48 82.55)
+    (descr "Circular Fiducial, 1mm bare copper top; 2mm keepout (Level A)")
+    (tags marker)
+    (attr virtual)
+    (fp_text reference REF** (at 0 -2) (layer F.SilkS) hide
+      (effects (font (size 1 1) (thickness 0.15)))
+    )
+    (fp_text value Fiducial_1mm_Dia_2mm_Outer (at 0 2) (layer F.Fab)
+      (effects (font (size 1 1) (thickness 0.15)))
+    )
+    (fp_circle (center 0 0) (end 1 0) (layer F.Fab) (width 0.1))
+    (fp_text user %R (at 0 0) (layer F.Fab)
+      (effects (font (size 0.4 0.4) (thickness 0.06)))
+    )
+    (fp_circle (center 0 0) (end 1.25 0) (layer F.CrtYd) (width 0.05))
+    (pad ~ smd circle (at 0 0) (size 1 1) (layers F.Cu F.Mask)
+      (solder_mask_margin 0.5) (clearance 0.5))
+  )
+  (module Fiducials:Fiducial_1mm_Dia_2mm_Outer (layer F.Cu)
+    (at 143.51 115.57)
+    (descr "Circular Fiducial, 1mm bare copper top; 2mm keepout (Level A)")
+    (tags marker)
+    (attr virtual)
+    (fp_text reference REF** (at 0 -2) (layer F.SilkS) hide
+      (effects (font (size 1 1) (thickness 0.15)))
+    )
+    (fp_text value Fiducial_1mm_Dia_2mm_Outer (at 0 2) (layer F.Fab)
+      (effects (font (size 1 1) (thickness 0.15)))
+    )
+    (fp_circle (center 0 0) (end 1 0) (layer F.Fab) (width 0.1))
+    (fp_text user %R (at 0 0) (layer F.Fab)
+      (effects (font (size 0.4 0.4) (thickness 0.06)))
+    )
+    (fp_circle (center 0 0) (end 1.25 0) (layer F.CrtYd) (width 0.05))
+    (pad ~ smd circle (at 0 0) (size 1 1) (layers F.Cu F.Mask)
+      (solder_mask_margin 0.5) (clearance 0.5))
+  )
   (module Mounting_Holes:MountingHole_3.2mm_M3 (layer F.Cu)
     (at 119.761 83.5025)
@@
     (pad 1 np_thru_hole circle (at 0 0) (size 3.2 3.2) (drill 3.2) (layers *.Cu *.Mask))
   )
+  (module Fiducials:Fiducial_1mm_Dia_2mm_Outer (layer F.Cu)
+    (at 129.54 82.55)
+    (descr "Circular Fiducial, 1mm bare copper top; 2mm keepout (Level A)")
+    (tags marker)
+    (attr virtual)
+    (fp_text reference REF** (at 0 -2) (layer F.SilkS) hide
+      (effects (font (size 1 1) (thickness 0.15)))
+    )
+    (fp_text value Fiducial_1mm_Dia_2mm_Outer (at 0 2) (layer F.Fab)
+      (effects (font (size 1 1) (thickness 0.15)))
+    )
+    (fp_circle (center 0 0) (end 1 0) (layer F.Fab) (width 0.1))
+    (fp_text user %R (at 0 0) (layer F.Fab)
+      (effects (font (size 0.4 0.4) (thickness 0.06)))
+    )
+    (fp_circle (center 0 0) (end 1.25 0) (layer F.CrtYd) (width 0.05))
+    (pad ~ smd circle (at 0 0) (size 1 1) (layers F.Cu F.Mask)
+      (solder_mask_margin 0.5) (clearance 0.5))
+  )
   (dimension 31.369 (width 0.3) (layer Dwgs.User)

Commit message: Lee Edits
Parts:
- moved D7 29.8 mm to (157.5, 86.5), turned to 270 degrees
- moved D4 25.7 mm to (151.1, 99.6)
- moved C3 25.3 mm to (168.3, 110.5), turned to 180 degrees
- moved D5 25.3 mm to (151.4, 93.7), turned to 270 degrees
- moved D2 24.4 mm to (154.3, 106.0), turned to 90 degrees
- moved C22 23.9 mm to (140.9, 106.7), turned to 0 degrees
- moved D6 23.7 mm to (154.3, 92.1), turned to 270 degrees
- moved U8 23.3 mm to (143.3, 110.5), turned to 0 degrees
- moved R1 21.5 mm to (168.3, 108.0), turned to 180 degrees
- moved D1 18.3 mm to (160.7, 108.0), turned to 90 degrees
- moved C21 16.3 mm to (126.5, 82.5), turned to 90 degrees
- moved C20 16.1 mm to (128.0, 82.2), turned to 90 degrees
- moved U7 16.0 mm to (132.1, 82.1)
- moved REF** 15.4 mm to (116.2, 90.2)
- moved C16 14.6 mm to (137.0, 83.2), turned to 180 degrees
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Connections:
- net +3.3VA renamed +3VA
- C3 pad 2: GND -> SHIELD_GND
- D1 pad 2: GND -> SHIELD_GND
- D2 pad 2: GND -> SHIELD_GND
- D3 pad 2: GND -> SHIELD_GND
- D4 pad 1: SCK_+ -> SCK_-
- D4 pad 2: GND -> SHIELD_GND
- D5 pad 1: SCK_- -> SCK_+
- D5 pad 2: GND -> SHIELD_GND
- D6 pad 1: CONVST_+ -> CONVST_-
- D6 pad 2: GND -> SHIELD_GND
- D7 pad 1: CONVST_- -> CONVST_+
- D7 pad 2: GND -> SHIELD_GND
- J1 pad 4: SCK_+ -> SCK_-
- J1 pad 5: SCK_- -> SCK_+
- J1 pad 7: CONVST_+ -> CONVST_-
- J1 pad 8: CONVST_- -> CONVST_+
- R1 pad 2: GND -> SHIELD_GND
- U9 pad 5: CONVST_- -> SCK_-
- U9 pad 6: CONVST_+ -> SCK_+
- U9 pad 7: SCK_- -> CONVST_-
- U9 pad 8: SCK_+ -> CONVST_+
Routing:
- net /MISO: track 35.6 -> 4.15 mm
- net SCK_-: track 32.4 -> 12.1 mm
- net SCK_+: track 34.7 -> 15.5 mm
- net MISO_-: track 33.2 -> 15.5 mm
- net SHIELD_GND: track 0.00 -> 17.1 mm, vias 0 -> 9
- net +5V: track 37.4 -> 52.8 mm, vias 0 -> 2
- net +3VA: track 31.1 -> 17.6 mm, vias 7 -> 6
- net CONVST_-: track 27.9 -> 15.5 mm
- net GND: track 71.3 -> 63.5 mm, vias 50 -> 40
- net MISO_+: track 28.5 -> 20.8 mm
- net CONVST_+: track 29.7 -> 22.4 mm
- net SCLK: track 35.2 -> 28.4 mm, vias 3 -> 2
- net Net-(C3-Pad1): track 25.0 -> 22.6 mm, vias 1 -> 0
- net CONVST: track 39.3 -> 38.5 mm, vias 3 -> 4
- net +3V3: track 39.4 -> 38.7 mm
- added copper zone on B.Cu, net SHIELD_GND
