File: Accelerometer/BELM_Accelerometer.sch (KiCad schematic (older format))
At the start: 3 parts

Commit message: First Rev to Review
Parts:
- added C10, C14, C15, C16, C8, C9: 1uF, symbol C
- added C11, C12, C13, C17, C18: 10uF, symbol C
- added C19: 0.1uF, symbol C
- added C3, C4, C5: 1nF, symbol C
- added C6, C7: 10nF, symbol C
- added D1, D2, D3, D4, D5: 6.8V, symbol D_Schottky_ALT
- added J1: CONN_01X10, symbol CONN_01X10
- added R1: 20, symbol R
- added U2: TSV914IPT, symbol TSV914IPT
- added U3, U4, U5: ADS8864, symbol ADS8864
- added U6: MAX6126B30+, symbol MAX6126B30+
- C1: renamed from C?; value C -> 10uF
- C2: renamed from C?; value C -> 0.1uF
- gave numbers to parts that had none: 1
Connections:
- net labels added: +3.3VA, +3V3, CONVST, MISO, MOSI, SCLK
- net labels removed: VDD
- wire segments 9 -> 144
- no-connect marks 0 -> 3
Other:
- note added: "Fc = 1.45uF/Cload\n"
- moved on the sheet: C1, C2, U1

Commit message: Rev 1
Other:
- note added: "3.3V Analog Reference"
- note added: "Connector To Shield"
Changed lines of the file:
@@
 Connection ~ 14900 2700
 Connection ~ 14900 2800
+Wire Notes Line
+	13100 1700 13100 3750
+Wire Notes Line
+	13100 3500 15750 3500
+Wire Notes Line
+	15750 1700 15750 3750
+Wire Notes Line
+	15750 1700 13100 1700
+Wire Notes Line
+	15750 3750 13100 3750
+Text Notes 13950 3650 0    60   ~ 0
+3.3V Analog Reference
+Wire Notes Line
+	13350 5600 13350 8100
+Wire Notes Line
+	13350 7750 16150 7750
+Wire Notes Line
+	16150 5450 16150 8100
+Wire Notes Line
+	16150 5450 13350 5450
+Wire Notes Line
+	13350 5450 13350 5650
+Wire Notes Line
+	16150 8100 13350 8100
+Text Notes 14350 7950 0    60   ~ 0
+Connector To Shield
 $EndSCHEMATC

Commit message: Update PCB
Parts:
- removed C4, C5: 1nF, symbol C
- removed C7: 10nF, symbol C
- added C? (x2): 1000pF, symbol C
- added C?: 10000pF, symbol C
- added R? (x3): 20, symbol R
- C?: renamed from C3; value 1nF -> 1000pF
- C?: renamed from C6; value 10nF -> 10000pF
- renumbered C1 to C?, C2 to C?, C10 to C?, C16 to C?, C13 to C?, C9 to C?, C15 to C?, C8 to C?, C14 to C?, C12 to C?, C11 to C?, C17 to C?, C18 to C?, C19 to C?, D5 to D?, D3 to D?, D1 to D?, D2 to D?, D4 to D?, J1 to J?, R1 to R?, U1 to U?, U2 to U?, U5 to U?, U4 to U?, U3 to U?, U6 to U?
Connections:
- wire segments 144 -> 147
Other:
- moved on the sheet: D?

Commit message: Updated
Parts:
- removed D? (x5): 6.8V, symbol D_Schottky_ALT
- removed J?: CONN_01X10, symbol CONN_01X10
- added C? (x2): 1uF, symbol C
- added D? (x3): 6.8V, symbol D_Schottky_ALT
- added J?: RJ45, symbol RJ45
- added U?: SN74AHC1G125, symbol SN74AHC1G125
- added U?: MIC5504-3.3, symbol MIC5504-3.3
- added U?: SN65LVDT390, symbol SN65LVDT390
Connections:
- net labels added: +5V, CONVST_+, CONVST_-, MISO_+, MISO_-, SCK_+, SCK_-
- net labels removed: MOSI
- wire segments 147 -> 168
- no-connect marks 3 -> 8
Other:
- note added: "5V to 3.3V LDO"
- note added: "Note: Line Driver/Bus Buffer"
- moved on the sheet: C?, R?, U?

Commit message: For Todd Tomorrow
Parts:
- removed R?: 20, symbol R
- removed U?: SN74AHC1G125, symbol SN74AHC1G125
- removed U?: SN65LVDT390, symbol SN65LVDT390
- added C? (x2): 0.1uF, symbol C
- added D? (x4): 6.8V, symbol D_Schottky_ALT
- added U?: SN65LVDT34D, symbol SN65LVDT34D
- added U?: DS90LV017ATMX/NOPB, symbol DS90LV017ATMX/NOPB
Connections:
- net +3V3: now also C?.1, C?.1, U?.1 (VCC), U?.1 (VCC)
- net CONVST: now also U?.2 (1Y); no longer U?.6 (CONVST)
- net CONVST_+: now also D?.1 (K), U?.7 (1B)
- net CONVST_-: now also D?.1 (K), U?.8 (1A)
- net GND: now also C?.2, C?.2, D?.2 (A), D?.2 (A), D?.2 (A), D?.2 (A), U?.4 (GND), U?.4 (GND)
- net MISO: now also U?.7 (DOUT), U?.2 (DI1)
- net MISO_+: now also U?.8 (DO1-)
- net MISO_-: now also U?.7 (DO1+)
- net SCK_+: now also D?.1 (K), U?.5 (2B)
- net SCK_-: now also D?.1 (K), U?.6 (2A)
- net SCLK: now also U?.3 (2Y); no longer U?.8 (SCLK)
- no-connect marks 8 -> 5
Other:
- note added: "LVDS Receiver"
- note added: "LVDS Transmitter"
- note removed: "Note: Line Driver/Bus Buffer"
- moved on the sheet: C?, D?, J?, R?, U?

Commit message: Todd's Revisions
Parts:
- removed C?: 10000pF, symbol C
- added C?: DNP, symbol C
- added R?: 0, symbol R
Connections:
- net +3.3VA: now also C?.1, C?.1, U?.14 (VDD), U?.15 (RES)
- net +3V3: no longer C?.1, C?.1, U?.14 (VDD), U?.15 (RES)
- net CONVST: now also U?.6 (CONVST), U?.9 (DIN)
- net CONVST_+: now also U?.8 (1A); no longer U?.7 (1B)
- net CONVST_-: now also U?.7 (1B); no longer U?.8 (1A)
- net GND: now also U?.11 (VCC-), U?.12 (In4+), U?.13 (In4-), U?.14 (OUT4), C?.2, R?.2; no longer U?.2 (In1-), U?.6 (In2-), U?.9 (In3-)
- net MISO_+: now also U?.7 (DO1+); no longer U?.8 (DO1-)
- net MISO_-: now also U?.8 (DO1-); no longer U?.7 (DO1+)
- net SCK_+: now also U?.6 (2A); no longer U?.5 (2B)
- net SCK_-: now also U?.5 (2B); no longer U?.6 (2A)
- net SCLK: now also U?.8 (SCLK)
- net at U?.1 (OUT1), U?.3 (AINP): now also U?.2 (In1-)
- net at U?.3 (AINP), U?.7 (Out2): now also U?.6 (In2-)
- net at U?.3 (AINP), U?.8 (Out3): now also U?.9 (In3-)
- net at J?.9 (SHIELD): now also C?.1, R?.1
- no-connect marks 5 -> 0

Commit message: Final Review
Parts:
- removed C? (x7): 1uF, symbol C
- removed C? (x5): 10uF, symbol C
- removed C? (x3): 0.1uF, symbol C
- removed C? (x2): 1000pF, symbol C
- removed R? (x2): 20, symbol R
- added C10, C11, C12, C17, C18, C19, C9: 1uF, Capacitors_SMD:C_0603, symbol C
- added C13, C14, C15, C16, C20: 10uF, Capacitors_SMD:C_0603, symbol C
- added C21, C22, C23: 0.1uF, Capacitors_SMD:C_0402, symbol C
- added C5, C6: 1000pF, Capacitors_SMD:C_0402, symbol C
- added R2, R3: 20, Resistors_SMD:R_0603, symbol R
- C1, C8: renamed from C?; footprint (none) -> Capacitors_SMD:C_0603; Voltage (none) -> 6.3V
- C2, C4, C7: renamed from C?; footprint (none) -> Capacitors_SMD:C_0402; Voltage (none) -> 6.3V
- C3: renamed from C?; footprint (none) -> Capacitors_SMD:C_0805; Voltage (none) -> 6.3V
- D1, D2, D3, D4, D5, D6, D7: renamed from D?; footprint (none) -> Senior_Design:SOD-123FL
- J1: renamed from J?; footprint (none) -> Senior_Design:A-2004-2-4-LPS-N-R
- R1: renamed from R?; footprint (none) -> Resistors_SMD:R_0805
- R4: renamed from R?; footprint (none) -> Resistors_SMD:R_0603
- U1: renamed from U?; footprint (none) -> Senior_Design:16-LGA
- U2: renamed from U?; footprint (none) -> TO_SOT_Packages_SMD:SOT-23-5
- U3: renamed from U?; footprint (none) -> Housings_SSOP:TSSOP-14_4.4x5mm_Pitch0.65mm
- U4, U5, U6: renamed from U?; footprint (none) -> Housings_SSOP:TSSOP-10_3x3mm_Pitch0.5mm
- U7: renamed from U?; footprint (none) -> Senior_Design:uMAX
- U8, U9: renamed from U?; footprint (none) -> Housings_SOIC:SOIC-8_3.9x4.9mm_Pitch1.27mm
Connections:
- net +3.3VA: now also C7.1, U3.4 (VCC+), C20.1, C21.1, R2.1, R3.1
- net +3V3: now also C10.2, C11.2, C12.2, C17.1, C18.1, C19.1, C22.1, C23.1, C9.1; no longer C7.1, U3.4 (VCC+)
- net CONVST: now also U9.3 (2Y); no longer U9.2 (1Y)
- net CONVST_+: now also U9.6 (2A); no longer U9.8 (1A)
- net CONVST_-: now also U9.5 (2B); no longer U9.7 (1B)
- net GND: now also C10.1, C11.1, C12.1, C13.2, C14.2, C15.2, C16.1, C17.2, C18.2, C19.2, C20.2, C21.2, C22.2, C23.2, C5.2, C6.2, C9.2
- net SCK_+: now also U9.8 (1A); no longer U9.6 (2A)
- net SCK_-: now also U9.7 (1B); no longer U9.5 (2B)
- net SCLK: now also U9.2 (1Y); no longer U9.3 (2Y)
- net Yout: now reaches U1.10 (Yout), U3.5 (In2+)
- net Yout: now also C5.1
- net Xout: now reaches C4.1, U1.12 (Xout), U3.3 (In1+)
- net Zout: now reaches U1.8 (Zout), U3.10 (In3+)
- net Zout: now also C6.1
- net at R4.2, U6.1 (REF): now also C15.1
- net at U5.1 (REF): now also C14.1, R3.2
- net at U4.1 (REF): now also C13.1, R2.2
- net at U7.1 (NR): now also C16.2
Other:
- moved on the sheet: D2, D3

Commit message: Lee Edits
Connections:
- net CONVST_+: now also D7.1 (K), J1.8, U9.8 (1A); no longer D6.1 (K), J1.7, U9.6 (2A)
- net CONVST_-: now also D6.1 (K), J1.7, U9.7 (1B); no longer D7.1 (K), J1.8, U9.5 (2B)
- net GND: no longer C3.2, D1.2 (A), D2.2 (A), D3.2 (A), D4.2 (A), D5.2 (A), D6.2 (A), D7.2 (A), R1.2
- net SCK_+: now also D5.1 (K), J1.5, U9.6 (2A); no longer D4.1 (K), J1.4, U9.8 (1A)
- net SCK_-: now also D4.1 (K), J1.4, U9.5 (2B); no longer D5.1 (K), J1.5, U9.7 (1B)
- net +3.3VA renamed +3VA
- new net SHIELD_GND: C3.2, D1.2 (A), D2.2 (A), D3.2 (A), D4.2 (A), D5.2 (A), D6.2 (A), D7.2 (A), R1.2
Other:
- note added: "3V Analog Reference"
- note removed: "3.3V Analog Reference"
- moved on the sheet: C3, D1, D2, D3, D4, D5, D6, D7, J1, R1
