File: Pi_Shield/RPi_Shield.sch (KiCad schematic (older format))
At the start: 5 parts

Commit message: Hello
Parts:
- added C? (x4): 0.1uF, symbol C
- added C? (x3): C, symbol C
- added D? (x36): D_Schottky_ALT, symbol D_Schottky_ALT
- added J? (x3): RJ45_2PORT, symbol RJ45_2PORT
- added R? (x3): R, symbol R
- added U? (x4): FIN1027AMX, symbol FIN1027AMX
Connections:
- net +3V3: now also C?.1, C?.1, C?.1, C?.1, U?.1 (VCC), U?.1 (VCC), U?.1 (VCC), U?.1 (VCC)
- net CONVST: now also U?.2 (DIN1)
- net GND: now also C?.2, C?.2, C?.2, C?.2, J?.1_6, J?.1_6, J?.1_6, J?.2_6, J?.2_6, J?.2_6, U?.4 (GND), U?.4 (GND), U?.4 (GND), U?.4 (GND)
- net ACCEL_0 renamed A0_SCK
- net A0_SCK: now also U?.2 (DIN1)
- net ACCEL_1 renamed A1_SCK
- net A1_SCK: now also U?.3 (DIN2)
- net ACCEL_2 renamed A2_SCK
- net A2_SCK: now also U?.2 (DIN1)
- net ACCEL_3 renamed A3_SCK
- net A3_SCK: now also U?.3 (DIN2)
- net ACCEL_4 renamed A4_SCK
- net A4_SCK: now also U?.2 (DIN1)
- net ACCEL_5 renamed A5_SCK
- net A5_SCK: now also U?.3 (DIN2)
- net SPI_MOSI_+ renamed SPI_MISO_+
- net SPI_MISO_+: now also D?.1 (K), D?.1 (K), D?.1 (K), D?.1 (K), D?.1 (K), D?.1 (K), J?.1_1, J?.1_1, J?.1_1, J?.2_1, J?.2_1, J?.2_1
- net SPI_MOSI_- renamed SPI_MISO_-
- net SPI_MISO_-: now also D?.1 (K), D?.1 (K), D?.1 (K), D?.1 (K), D?.1 (K), D?.1 (K), J?.1_2, J?.1_2, J?.1_2, J?.2_2, J?.2_2, J?.2_2
- new net: C?.1, J?.9 (SHIELD), R?.1 (x3)
- new net +5V: J?.1_3, J?.1_3, J?.1_3, J?.2_3, J?.2_3, J?.2_3
- new net A0_SCK+: D?.1 (K), J?.1_5, U?.8 (DOUT2-)
- new net A0_SCK-: D?.1 (K), J?.1_4, U?.8 (DOUT2-)
- new net A1_SCK+: D?.1 (K), J?.2_5, U?.8 (DOUT2-)
- new net A1_SCK-: D?.1 (K), J?.2_4, U?.8 (DOUT2-)
- new net A2_SCK+: D?.1 (K), J?.1_5, U?.8 (DOUT2-)
- new net A2_SCK-: D?.1 (K), J?.1_4, U?.8 (DOUT2-)
- new net A3_SCK+: D?.1 (K), J?.2_5, U?.8 (DOUT2-)
- new net A3_SCK-: D?.1 (K), J?.2_4, U?.8 (DOUT2-)
- new net A4_SCK+: D?.1 (K), J?.1_5, U?.8 (DOUT2-)
- new net A4_SCK-: D?.1 (K), J?.1_4, U?.8 (DOUT2-)
- new net A5_SCK+: D?.1 (K), J?.2_5, U?.8 (DOUT2-)
- new net A5_SCK-: D?.1 (K), J?.2_4, U?.8 (DOUT2-)
- new net CONVST+: D?.1 (K), D?.1 (K), D?.1 (K), D?.1 (K), D?.1 (K), D?.1 (K), J?.1_8, J?.1_8, J?.1_8, J?.2_8, J?.2_8, J?.2_8, U?.8 (DOUT2-)
- new net CONVST-: D?.1 (K), D?.1 (K), D?.1 (K), D?.1 (K), D?.1 (K), D?.1 (K), J?.1_7, J?.1_7, J?.1_7, J?.2_7, J?.2_7, J?.2_7, U?.8 (DOUT2-)
- new net SHIELD_GND1: C?.2, D?.2 (A), D?.2 (A), D?.2 (A), D?.2 (A), D?.2 (A), D?.2 (A), D?.2 (A), D?.2 (A), D?.2 (A), D?.2 (A), D?.2 (A), D?.2 (A), R?.2
- new net SHIELD_GND2: C?.2, D?.2 (A), D?.2 (A), D?.2 (A), D?.2 (A), D?.2 (A), D?.2 (A), D?.2 (A), D?.2 (A), D?.2 (A), D?.2 (A), D?.2 (A), D?.2 (A), R?.2
- new net SHIELD_GND3: C?.2, D?.2 (A), D?.2 (A), D?.2 (A), D?.2 (A), D?.2 (A), D?.2 (A), D?.2 (A), D?.2 (A), D?.2 (A), D?.2 (A), D?.2 (A), D?.2 (A), R?.2
- no-connect marks 23 -> 26
Other:
- moved on the sheet: C?, J?, U?
